Commit message: arena done, martial club lil left

File: 2026_field.urdf (robot description, URDF)
Before this commit: robot robocon_2026_field_dual_rotated_forest, 45 links, 44 joints
Links:
- removed link line_arena_hor
- removed link line_arena_perp
- removed link platform_flat
- removed link platform_incline
- added link arena_border_front; visual box size=0.05 9.05 0.4
- added link b_line_arena_hor; visual box size=0.03 1.2 0
- added link b_line_arena_perp; visual box size=1.450 0.03 0
- added link elevated_plane_blue; visual box size=2.5 4.5 0
- added link elevated_plane_red; visual box size=2.5 4.5 0
- added link elevated_retry_blue; visual box size=1 1 0
- added link elevated_retry_red; visual box size=1 1 0
- added link elevated_small_blue; visual box size=1.2 1.5 0
- added link elevated_small_red; visual box size=1.2 1.5 0
- added link r_line_arena_hor; visual box size=0.03 1.2 0
- added link r_line_arena_perp; visual box size=1.450 0.03 0
- added link ramp_blue; visual box size=1.45 1.5 0
- added link ramp_red; visual box size=1.45 1.5 0
- added link tictac_base_link; visual box size=1.620 0.320 0.480
- added link tictac_hor_bottom; visual box size=1.660 0.320 0.02
- added link tictac_hor_top; visual box size=1.660 0.320 0.02
- added link tictac_middle_left; visual box size=0.02 0.320 1.540
- added link tictac_middle_right; visual box size=0.02 0.320 1.540
- added link tictac_side_left; visual box size=0.02 0.320 1.540
- added link tictac_side_right; visual box size=0.02 0.320 1.540
- added link tictac_top; visual box size=1.660 0.320 0.02
- link border_x_neg: geometry visual box size=0.05 12.0 0.500
Joints:
- removed joint line_arena_hor
- removed joint line_arena_perp
- removed joint platform_flat_joint
- removed joint platform_incline_joint
- added joint arena_border_front: type fixed, parent world, child arena_border_front, origin xyz=0 0 0 rpy=0 0 0
- added joint b_line_arena_hor: type fixed, parent world, child b_line_arena_hor, origin xyz=0 0 0 rpy=0 0 0
- added joint b_line_arena_perp: type fixed, parent world, child b_line_arena_perp, origin xyz=0 0 0 rpy=0 0 0
- added joint elevated_plane_blue: type fixed, parent world, child elevated_plane_blue, origin xyz=0 0 0 rpy=0 0 0
- added joint elevated_plane_red: type fixed, parent world, child elevated_plane_red, origin xyz=0 0 0 rpy=0 0 0
- added joint elevated_retry_blue: type fixed, parent world, child elevated_retry_blue, origin xyz=0 0 0 rpy=0 0 0
- added joint elevated_retry_red: type fixed, parent world, child elevated_retry_red, origin xyz=0 0 0 rpy=0 0 0
- added joint elevated_small_blue: type fixed, parent world, child elevated_small_blue, origin xyz=0 0 0 rpy=0 0 0
- added joint elevated_small_red: type fixed, parent world, child elevated_small_red, origin xyz=0 0 0 rpy=0 0 0
- added joint r_line_arena_hor: type fixed, parent world, child r_line_arena_hor, origin xyz=0 0 0 rpy=0 0 0
- added joint r_line_arena_perp: type fixed, parent world, child r_line_arena_perp, origin xyz=0 0 0 rpy=0 0 0
- added joint ramp_blue: type fixed, parent world, child ramp_blue, origin xyz=0 0 0 rpy=0 0 0
- added joint ramp_red: type fixed, parent world, child ramp_red, origin xyz=0 0 0 rpy=0 0 0
- added joint tictac_base_link: type fixed, parent world, child tictac_base_link, origin xyz=0 0 0 rpy=0 0 0
- added joint tictac_hor_bottom: type fixed, parent world, child tictac_hor_bottom, origin xyz=0 0 0 rpy=0 0 0
- added joint tictac_hor_top: type fixed, parent world, child tictac_hor_top, origin xyz=0 0 0 rpy=0 0 0
- added joint tictac_middle_left: type fixed, parent world, child tictac_middle_left, origin xyz=0 0 0 rpy=0 0 0
- added joint tictac_middle_right: type fixed, parent world, child tictac_middle_right, origin xyz=0 0 0 rpy=0 0 0
- added joint tictac_side_left: type fixed, parent world, child tictac_side_left, origin xyz=0 0 0 rpy=0 0 0
- added joint tictac_side_right: type fixed, parent world, child tictac_side_right, origin xyz=0 0 0 rpy=0 0 0
- added joint tictac_top: type fixed, parent world, child tictac_top, origin xyz=0 0 0 rpy=0 0 0

Commit message: Field design Complete

File: 2026_field.urdf (robot description, URDF)
Before this commit: robot robocon_2026_field_dual_rotated_forest, 62 links, 61 joints
Links:
- added link auto_start_blue; visual box size=0.8 0.8 0.001
- added link auto_start_red; visual box size=0.8 0.8 0.001
- added link border_neg_y_pos_hidden; visual box size=1.5 0.05 0.40
- added link border_y_neg_big; visual box size=2.550 0.05 0.50
- added link border_y_pos_big; visual box size=2.550 0.05 0.50
- added link border_y_pos_hidden; visual box size=1.5 0.05 0.40
- added link spear_head_rack; visual box size=1.2 0.3 0.50
- added link staff_blue; visual box size=0.3 0.8 0.5
- added link staff_red; visual box size=0.3 0.8 0.5
Joints:
- added joint auto_start_blue: type fixed, parent world, child auto_start_blue, origin xyz=0 0 0 rpy=0 0 0
- added joint auto_start_red: type fixed, parent world, child auto_start_red, origin xyz=0 0 0 rpy=0 0 0
- added joint border_neg_y_pos_hidden: type fixed, parent world, child border_neg_y_pos_hidden, origin xyz=0 0 0
- added joint border_y_neg_joint_big: type fixed, parent world, child border_y_neg_big, origin xyz=0 0 0
- added joint border_y_pos_hidden: type fixed, parent world, child border_y_pos_hidden, origin xyz=0 0 0
- added joint border_y_pos_joint_big: type fixed, parent world, child border_y_pos_big, origin xyz=0 0 0
- added joint spear_head_rack: type fixed, parent world, child spear_head_rack, origin xyz=0 0 0 rpy=0 0 0
- added joint staff_blue: type fixed, parent world, child staff_blue, origin xyz=0 0 0 rpy=0 0 0
- added joint staff_red: type fixed, parent world, child staff_red, origin xyz=0 0 0 rpy=0 0 0

Commit message: Successfully opened in Gazebo

File: 2026_field.urdf (robot description, URDF)
Before this commit: robot robocon_2026_field_dual_rotated_forest, 71 links, 70 joints
Links:
- removed link world
- added link base_link
- added link yellow_blue, mass 0.1; collision box size=0.3 1.4 0.001; visual box size=0.3 1.4 0.001
- added link yellow_red, mass 0.1; collision box size=0.3 1.4 0.001; visual box size=0.3 1.4 0.001
- link arena_border_front: mass None -> 1.5; geometry collision box size=0.05 9.05 0.4; visual box size=0.05 9.05 0.4
- link auto_start_blue: mass None -> 0.5; geometry collision box size=0.8 0.8 0.001; visual box size=0.8 0.8 0.001
- link auto_start_red: mass None -> 0.5; geometry collision box size=0.8 0.8 0.001; visual box size=0.8 0.8 0.001
- link b_line_arena_hor: mass None -> 0.05; geometry collision box size=0.03 1.2 0.001; visual box size=0.03 1.2 0.001
- link b_line_arena_perp: mass None -> 0.05; geometry collision box size=1.45 0.03 0.001; visual box size=1.45 0.03 0.001
- link b_line_martial_perp1: mass None -> 0.05; geometry collision box size=1.215 0.03 0.001; visual box size=1.215 0.03 0.001
- link b_line_martial_perp2: mass None -> 0.05; geometry collision box size=1.215 0.03 0.001; visual box size=1.215 0.03 0.001
- link b_r1_c1: mass None -> 1.0; geometry collision box size=1.20 1.20 0.20; visual box size=1.20 1.20 0.20
- link b_r1_c2: mass None -> 1.0; geometry collision box size=1.20 1.20 0.40; visual box size=1.20 1.20 0.40
- link b_r1_c3: mass None -> 1.0; geometry collision box size=1.20 1.20 0.20; visual box size=1.20 1.20 0.20
- link b_r2_c1: mass None -> 1.0; geometry collision box size=1.20 1.20 0.40; visual box size=1.20 1.20 0.40
- link b_r2_c2: mass None -> 1.0; geometry collision box size=1.20 1.20 0.60; visual box size=1.20 1.20 0.60
- link b_r2_c3: mass None -> 1.0; geometry collision box size=1.20 1.20 0.40; visual box size=1.20 1.20 0.40
- link b_r3_c1: mass None -> 1.0; geometry collision box size=1.20 1.20 0.20; visual box size=1.20 1.20 0.20
- link b_r3_c2: mass None -> 1.0; geometry collision box size=1.20 1.20 0.40; visual box size=1.20 1.20 0.40
- link b_r3_c3: mass None -> 1.0; geometry collision box size=1.20 1.20 0.60; visual box size=1.20 1.20 0.60
- link b_r4_c1: mass None -> 1.0; geometry collision box size=1.20 1.20 0.40; visual box size=1.20 1.20 0.40
- link b_r4_c2: mass None -> 1.0; geometry collision box size=1.20 1.20 0.20; visual box size=1.20 1.20 0.20
- link b_r4_c3: mass None -> 1.0; geometry collision box size=1.20 1.20 0.40; visual box size=1.20 1.20 0.40
- link blue_forest_base: mass None -> 0.1
- link border_neg_y_pos_hidden: mass None -> 0.5; geometry collision box size=1.5 0.05 0.40; visual box size=1.5 0.05 0.40
- link border_x_neg: mass None -> 2.0; geometry collision box size=0.05 12.0 0.500; visual box size=0.05 12.0 0.500
- link border_x_pos: mass None -> 1.0; geometry collision box size=0.05 12.0 0.10; visual box size=0.05 12.0 0.10
- link border_y_neg: mass None -> 1.0; geometry collision box size=12.0 0.05 0.10; visual box size=12.0 0.05 0.10
- link border_y_neg_big: mass None -> 1.0; geometry collision box size=2.550 0.05 0.50; visual box size=2.550 0.05 0.50
- link border_y_pos: mass None -> 1.0; geometry collision box size=12.0 0.05 0.10; visual box size=12.0 0.05 0.10
- link border_y_pos_big: mass None -> 1.0; geometry collision box size=2.550 0.05 0.50; visual box size=2.550 0.05 0.50
- link border_y_pos_hidden: mass None -> 0.5; geometry collision box size=1.5 0.05 0.40; visual box size=1.5 0.05 0.40
- link elevated_plane_blue: mass None -> 5.0; geometry collision box size=2.5 4.5 0.001; visual box size=2.5 4.5 0.001
- link elevated_plane_red: mass None -> 5.0; geometry collision box size=2.5 4.5 0.001; visual box size=2.5 4.5 0.001
- link elevated_retry_blue: mass None -> 0.2; geometry collision box size=1 1 0.001; visual box size=1 1 0.001
- link elevated_retry_red: mass None -> 0.2; geometry collision box size=1 1 0.001; visual box size=1 1 0.001
- link elevated_small_blue: mass None -> 1.0; geometry collision box size=1.2 1.5 0.001; visual box size=1.2 1.5 0.001
- link elevated_small_red: mass None -> 1.0; geometry collision box size=1.2 1.5 0.001; visual box size=1.2 1.5 0.001
- link internal_divider: mass None -> 1.0; geometry collision box size=12.0 0.05 0.10; visual box size=12.0 0.05 0.10
- link left_field_surface: mass None -> 10.0; geometry collision box size=12.0 6.0 0.001; visual box size=12.0 6.0 0.001
- link line_martial: mass None -> 0.1; geometry collision box size=0.03 12.0 0.001; visual box size=0.03 12.0 0.001
- link manual_start_blue: mass None -> 0.5; geometry collision box size=1 1 0.001; visual box size=1 1 0.001
- link manual_start_red: mass None -> 0.5; geometry collision box size=1 1 0.001; visual box size=1 1 0.001
- link r_line_arena_hor: mass None -> 0.05; geometry collision box size=0.03 1.2 0.001; visual box size=0.03 1.2 0.001
- link r_line_arena_perp: mass None -> 0.05; geometry collision box size=1.45 0.03 0.001; visual box size=1.45 0.03 0.001
- link r_line_martial_perp1: mass None -> 0.05; geometry collision box size=1.215 0.03 0.001; visual box size=1.215 0.03 0.001
- link r_line_martial_perp2: mass None -> 0.05; geometry collision box size=1.215 0.03 0.001; visual box size=1.215 0.03 0.001
- link r_r1_c1: mass None -> 1.0; geometry collision box size=1.20 1.20 0.20; visual box size=1.20 1.20 0.20
- link r_r1_c2: mass None -> 1.0; geometry collision box size=1.20 1.20 0.40; visual box size=1.20 1.20 0.40
- link r_r1_c3: mass None -> 1.0; geometry collision box size=1.20 1.20 0.20; visual box size=1.20 1.20 0.20
- link r_r2_c1: mass None -> 1.0; geometry collision box size=1.20 1.20 0.40; visual box size=1.20 1.20 0.40
- link r_r2_c2: mass None -> 1.0; geometry collision box size=1.20 1.20 0.60; visual box size=1.20 1.20 0.60
- link r_r2_c3: mass None -> 1.0; geometry collision box size=1.20 1.20 0.40; visual box size=1.20 1.20 0.40
- link r_r3_c1: mass None -> 1.0; geometry collision box size=1.20 1.20 0.60; visual box size=1.20 1.20 0.60
- link r_r3_c2: mass None -> 1.0; geometry collision box size=1.20 1.20 0.40; visual box size=1.20 1.20 0.40
- link r_r3_c3: mass None -> 1.0; geometry collision box size=1.20 1.20 0.60; visual box size=1.20 1.20 0.60
- link r_r4_c1: mass None -> 1.0; geometry collision box size=1.20 1.20 0.40; visual box size=1.20 1.20 0.40
- link r_r4_c2: mass None -> 1.0; geometry collision box size=1.20 1.20 0.20; visual box size=1.20 1.20 0.20
- link r_r4_c3: mass None -> 1.0; geometry collision box size=1.20 1.20 0.40; visual box size=1.20 1.20 0.40
- link ramp_blue: mass None -> 1.0; geometry collision box size=1.45 1.5 0.01; visual box size=1.45 1.5 0.01
- link ramp_red: mass None -> 1.0; geometry collision box size=1.45 1.5 0.01; visual box size=1.45 1.5 0.01
- link red_forest_base: mass None -> 0.1
- link right_field_surface: mass None -> 10.0; geometry collision box size=12.0 6.0 0.001; visual box size=12.0 6.0 0.001
- link spear_head_rack: mass None -> 1.0; geometry collision box size=1.2 0.3 0.50; visual box size=1.2 0.3 0.50
- link staff_blue: mass None -> 0.5; geometry collision box size=0.3 0.8 0.5; visual box size=0.3 0.8 0.5
- link staff_red: mass None -> 0.5; geometry collision box size=0.3 0.8 0.5; visual box size=0.3 0.8 0.5
- link tictac_base_link: mass None -> 3.0; geometry collision box size=1.62 0.32 0.48; visual box size=1.62 0.32 0.48
- link tictac_hor_bottom: mass None -> 0.2; geometry collision box size=1.66 0.32 0.02; visual box size=1.66 0.32 0.02
- link tictac_hor_top: mass None -> 0.2; geometry collision box size=1.66 0.32 0.02; visual box size=1.66 0.32 0.02
- link tictac_middle_left: mass None -> 0.5; geometry collision box size=0.02 0.32 1.54; visual box size=0.02 0.32 1.54
- link tictac_middle_right: mass None -> 0.5; geometry collision box size=0.02 0.32 1.54; visual box size=0.02 0.32 1.54
- link tictac_side_left: mass None -> 0.5; geometry collision box size=0.02 0.32 1.54; visual box size=0.02 0.32 1.54
- link tictac_side_right: mass None -> 0.5; geometry collision box size=0.02 0.32 1.54; visual box size=0.02 0.32 1.54
- link tictac_top: mass None -> 0.5; geometry collision box size=1.66 0.32 0.02; visual box size=1.66 0.32 0.02
Joints:
- removed joint arena_border_front
- removed joint auto_start_blue
- removed joint auto_start_red
- removed joint b_line_arena_hor
- removed joint b_line_arena_perp
- removed joint b_line_martial_perp1
- removed joint b_line_martial_perp2
- removed joint b_r1_c1_joint
- removed joint b_r1_c2_joint
- removed joint b_r1_c3_joint
- removed joint b_r2_c1_joint
- removed joint b_r2_c2_joint
- removed joint b_r2_c3_joint
- removed joint b_r3_c1_joint
- removed joint b_r3_c2_joint
- removed joint b_r3_c3_joint
- removed joint b_r4_c1_joint
- removed joint b_r4_c2_joint
- removed joint b_r4_c3_joint
- removed joint border_neg_y_pos_hidden
- removed joint border_y_pos_hidden
- removed joint elevated_plane_blue
- removed joint elevated_plane_red
- removed joint elevated_retry_blue
- removed joint elevated_retry_red
- removed joint elevated_small_blue
- removed joint elevated_small_red
- removed joint line_martial
- removed joint manual_start_blue
- removed joint manual_start_red
- removed joint r_line_arena_hor
- removed joint r_line_arena_perp
- removed joint r_line_martial_perp1
- removed joint r_line_martial_perp2
- removed joint r_r1_c1_joint
- removed joint r_r1_c2_joint
- removed joint r_r1_c3_joint
- removed joint r_r2_c1_joint
- removed joint r_r2_c2_joint
- removed joint r_r2_c3_joint
- removed joint r_r3_c1_joint
- removed joint r_r3_c2_joint
- removed joint r_r3_c3_joint
- removed joint r_r4_c1_joint
- removed joint r_r4_c2_joint
- removed joint r_r4_c3_joint
- removed joint ramp_blue
- removed joint ramp_red
- removed joint spear_head_rack
- removed joint staff_blue
- removed joint staff_red
- removed joint tictac_base_link
- removed joint tictac_hor_bottom
- removed joint tictac_hor_top
- removed joint tictac_middle_left
- removed joint tictac_middle_right
- removed joint tictac_side_left
- removed joint tictac_side_right
- removed joint tictac_top
- removed joint world_joint_blue_forest
- removed joint world_joint_red_forest
- added joint arena_border_front_joint: type fixed, parent base_link, child arena_border_front
- added joint auto_start_blue_joint: type fixed, parent base_link, child auto_start_blue
- added joint auto_start_red_joint: type fixed, parent base_link, child auto_start_red
- added joint b_line_arena_hor_joint: type fixed, parent base_link, child b_line_arena_hor
- added joint b_line_arena_perp_joint: type fixed, parent base_link, child b_line_arena_perp
- added joint b_line_martial_perp1_joint: type fixed, parent base_link, child b_line_martial_perp1
- added joint b_line_martial_perp2_joint: type fixed, parent base_link, child b_line_martial_perp2
- added joint base_link_joint_blue_forest: type fixed, parent base_link, child blue_forest_base, origin xyz=0.392 -4.8 0 rpy=0 0 1.5708
- added joint base_link_joint_red_forest: type fixed, parent base_link, child red_forest_base, origin xyz=0.392 1.2 0 rpy=0 0 1.5708
- added joint border_neg_y_pos_hidden_joint: type fixed, parent base_link, child border_neg_y_pos_hidden
- added joint border_y_pos_hidden_joint: type fixed, parent base_link, child border_y_pos_hidden
- added joint elevated_plane_blue_joint: type fixed, parent base_link, child elevated_plane_blue
- added joint elevated_plane_red_joint: type fixed, parent base_link, child elevated_plane_red
- added joint elevated_retry_blue_joint: type fixed, parent base_link, child elevated_retry_blue
- added joint elevated_retry_red_joint: type fixed, parent base_link, child elevated_retry_red
- added joint elevated_small_blue_joint: type fixed, parent base_link, child elevated_small_blue
- added joint elevated_small_red_joint: type fixed, parent base_link, child elevated_small_red
- added joint joint_b_r1_c1: type fixed, parent blue_forest_base, child b_r1_c1, origin xyz=0.60 1.80 0
- added joint joint_b_r1_c2: type fixed, parent blue_forest_base, child b_r1_c2, origin xyz=1.80 1.80 0
- added joint joint_b_r1_c3: type fixed, parent blue_forest_base, child b_r1_c3, origin xyz=3.00 1.80 0
- added joint joint_b_r2_c1: type fixed, parent blue_forest_base, child b_r2_c1, origin xyz=0.60 0.60 0
- added joint joint_b_r2_c2: type fixed, parent blue_forest_base, child b_r2_c2, origin xyz=1.80 0.60 0
- added joint joint_b_r2_c3: type fixed, parent blue_forest_base, child b_r2_c3, origin xyz=3.00 0.60 0
- added joint joint_b_r3_c1: type fixed, parent blue_forest_base, child b_r3_c1, origin xyz=0.60 -0.60 0
- added joint joint_b_r3_c2: type fixed, parent blue_forest_base, child b_r3_c2, origin xyz=1.80 -0.60 0
- added joint joint_b_r3_c3: type fixed, parent blue_forest_base, child b_r3_c3, origin xyz=3.00 -0.60 0
- added joint joint_b_r4_c1: type fixed, parent blue_forest_base, child b_r4_c1, origin xyz=0.60 -1.80 0
- added joint joint_b_r4_c2: type fixed, parent blue_forest_base, child b_r4_c2, origin xyz=1.80 -1.80 0
- added joint joint_b_r4_c3: type fixed, parent blue_forest_base, child b_r4_c3, origin xyz=3.00 -1.80 0
- added joint joint_r_r1_c1: type fixed, parent red_forest_base, child r_r1_c1, origin xyz=0.60 1.80 0
- added joint joint_r_r1_c2: type fixed, parent red_forest_base, child r_r1_c2, origin xyz=1.80 1.80 0
- added joint joint_r_r1_c3: type fixed, parent red_forest_base, child r_r1_c3, origin xyz=3.00 1.80 0
- added joint joint_r_r2_c1: type fixed, parent red_forest_base, child r_r2_c1, origin xyz=0.60 0.60 0
- added joint joint_r_r2_c2: type fixed, parent red_forest_base, child r_r2_c2, origin xyz=1.80 0.60 0
- added joint joint_r_r2_c3: type fixed, parent red_forest_base, child r_r2_c3, origin xyz=3.00 0.60 0
- added joint joint_r_r3_c1: type fixed, parent red_forest_base, child r_r3_c1, origin xyz=0.60 -0.60 0
- added joint joint_r_r3_c2: type fixed, parent red_forest_base, child r_r3_c2, origin xyz=1.80 -0.60 0
- added joint joint_r_r3_c3: type fixed, parent red_forest_base, child r_r3_c3, origin xyz=3.00 -0.60 0
- added joint joint_r_r4_c1: type fixed, parent red_forest_base, child r_r4_c1, origin xyz=0.60 -1.80 0
- added joint joint_r_r4_c2: type fixed, parent red_forest_base, child r_r4_c2, origin xyz=1.80 -1.80 0
- added joint joint_r_r4_c3: type fixed, parent red_forest_base, child r_r4_c3, origin xyz=3.00 -1.80 0
- added joint line_martial_joint: type fixed, parent base_link, child line_martial
- added joint manual_start_blue_joint: type fixed, parent base_link, child manual_start_blue
- added joint manual_start_red_joint: type fixed, parent base_link, child manual_start_red
- added joint r_line_arena_hor_joint: type fixed, parent base_link, child r_line_arena_hor
- added joint r_line_arena_perp_joint: type fixed, parent base_link, child r_line_arena_perp
- added joint r_line_martial_perp1_joint: type fixed, parent base_link, child r_line_martial_perp1
- added joint r_line_martial_perp2_joint: type fixed, parent base_link, child r_line_martial_perp2
- added joint ramp_blue_joint: type fixed, parent base_link, child ramp_blue
- added joint ramp_red_joint: type fixed, parent base_link, child ramp_red
- added joint spear_head_rack_joint: type fixed, parent base_link, child spear_head_rack
- added joint staff_blue_joint: type fixed, parent base_link, child staff_blue
- added joint staff_red_joint: type fixed, parent base_link, child staff_red
- added joint tictac_base_link_joint: type fixed, parent base_link, child tictac_base_link
- added joint tictac_hor_bottom_joint: type fixed, parent base_link, child tictac_hor_bottom
- added joint tictac_hor_top_joint: type fixed, parent base_link, child tictac_hor_top
- added joint tictac_middle_left_joint: type fixed, parent base_link, child tictac_middle_left
- added joint tictac_middle_right_joint: type fixed, parent base_link, child tictac_middle_right
- added joint tictac_side_left_joint: type fixed, parent base_link, child tictac_side_left
- added joint tictac_side_right_joint: type fixed, parent base_link, child tictac_side_right
- added joint tictac_top_joint: type fixed, parent base_link, child tictac_top
- added joint yellow_blue_joint: type fixed, parent base_link, child yellow_blue
- added joint yellow_red_joint: type fixed, parent base_link, child yellow_red
- joint border_x_neg_joint: origin xyz=0 0 0 -> (none); parent world -> base_link
- joint border_x_pos_joint: origin xyz=0 0 0 -> (none); parent world -> base_link
- joint border_y_neg_joint: origin xyz=0 0 0 -> (none); parent world -> base_link
- joint border_y_neg_joint_big: origin xyz=0 0 0 -> (none); parent world -> base_link
- joint border_y_pos_joint: origin xyz=0 0 0 -> (none); parent world -> base_link
- joint border_y_pos_joint_big: origin xyz=0 0 0 -> (none); parent world -> base_link
- joint internal_divider_joint: origin xyz=0 0 0 -> (none); parent world -> base_link
- joint left_field_joint: parent world -> base_link
- joint right_field_joint: parent world -> base_link
